File: HARDWARE/NeuroBytes-v091.kicad_pcb (KiCad board)
At the start: 2 copper layers, 56.4 x 30.9 mm, 55 parts, among them IC1 LD2980ABM50TR, IC2 ATTINY88-MM, P1 JST GH 4-position, P2 JST GH 4-position, P28 JST GH 4-position, P29 JST GH 4-position, P3 JST GH 4-position, P4 JST GH 4-position, P5 JST GH 4-position, SW1 SW_PUSH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

Commit message: added PCB and schematic screenshots
Parts:
- G***: moved to F.Cu
Changed lines of the file:
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@@
-(kicad_pcb (version 4) (host pcbnew 4.0.2-4+6225~38~ubuntu14.04.1-stable)
+(kicad_pcb (version 4) (host pcbnew 4.0.4+e1-6308~48~ubuntu14.04.1-stable)
   (general
     (links 109)
     (no_connects 12)
-    (area 29.85 69.5 117.22143 145.4)
+    (area 30 69.8 117.07143 146)
     (thickness 1.6)
     (drawings 187)
@@
   )
   (layers
-    (0 F.Cu signal)
+    (0 F.Cu signal hide)
     (31 B.Cu signal)
     (32 B.Adhes user)
-    (33 F.Adhes user)
-    (34 B.Paste user)
-    (35 F.Paste user hide)
+    (33 F.Adhes user hide)
+    (34 B.Paste user hide)
+    (35 F.Paste user)
     (36 B.SilkS user)
     (37 F.SilkS user hide)
@@
     (39 F.Mask user hide)
     (40 Dwgs.User user)
-    (41 Cmts.User user)
+    (41 Cmts.User user hide)
     (42 Eco1.User user)
     (43 Eco2.User user)
@@
     (46 B.CrtYd user)
     (47 F.CrtYd user)
-    (48 B.Fab user)
-    (49 F.Fab user)
+    (48 B.Fab user hide)
+    (49 F.Fab user hide)
   )
   (setup
@@
     (aux_axis_origin 39 113)
     (grid_origin 39 113)
-    (visible_elements FFFFFF3F)
+    (visible_elements FFFDD43F)
     (pcbplotparams
-      (layerselection 0x210fc_80000001)
+      (layerselection 0x310fc_80000001)
       (usegerberextensions false)
       (excludeedgelayer true)
@@
       (net 1 GND))
   )
-  (module NeuroBytes-v09:v09-logo-fmask (layer F.Mask)
+  (module NeuroBytes-v09:v09-logo-fmask (layer F.Cu)
     (at 66.44 99.1)
     (fp_text reference G*** (at 0 0) (layer F.SilkS) hide
